File: out/cv-module.kicad_sch (KiCad schematic)
At the start: 238 parts, among them J1 CH1, J10 CTRL2, J11 CTRL3, J2 CH2, J3 CH3, J4 CH4, J5 CH5, J6 CH6, J7 BOND, J8 PWR, J9 CTRL, K801 DPDT, K802 DPDT, K803 DPDT, Q801 DMG1012T, U1 OPA1644, U10 SSI2164, U11 74AHC541, U12 MAX6126A25, U13 TL074, U14 TL074, U15 TMR6-2422WI, U16 NCP1117-5.0, U2 OPA1644, U3 OPA1644, U4 OPA1644, U5 OPA1644, U6 OPA1644, U7 OPA1644, U8 OPA1644, U9 SSI2164

Commit message: choke and adc
Parts:
- added C152, C252, C352, C452, C552, C652: 1200p/50V C0G, Capacitor_SMD:C_0805_2012Metric, symbol Device:C
- added C815, C816: 1u/16V X7R, Capacitor_SMD:C_0805_2012Metric, symbol Device:C
- added C817, C818, C819: 100n/50V X7R, Capacitor_SMD:C_0805_2012Metric, symbol Device:C
- added J12: SPI, Connector_PinHeader_2.54mm:PinHeader_1x05_P2.54mm_Vertical, symbol Connector_Generic:Conn_01x05
- added J13: SPI2, Connector_PinHeader_2.54mm:PinHeader_1x05_P2.54mm_Vertical, symbol Connector_Generic:Conn_01x05
- added L801: 744222, Inductor_SMD:L_CommonMode_Wuerth_WE-SL2, symbol cv:744222
- added R156, R256, R356, R456, R556, R656: 22k 1%, Resistor_SMD:R_0805_2012Metric, symbol Device:R
- added R157, R257, R357, R457, R557, R657: 4k99 1%, Resistor_SMD:R_0805_2012Metric, symbol Device:R
- added U17: MCP3564, Package_SO:TSSOP-20_4.4x6.5mm_P0.65mm, symbol cv:MCP3564
- added U18: MCP1700-3.3, Package_TO_SOT_SMD:SOT-23, symbol cv:MCP1700-3.3
Connections:
- net ENV1: now also R156.1
- net ENV2: now also R256.1
- net ENV3: now also R356.1
- net ENV4: now also R456.1
- net ENV5: now also R556.1
- net ENV6: now also R656.1
- net IGND: now also L801.3; no longer J8.2 (Pin_2)
- net MAGND: now also C152.2, C252.2, C352.2, C452.2, C552.2, C652.2, C815.2, C816.2, C817.2, C818.2, C819.2, R157.2, R257.2, R357.2, R457.2, R557.2, R657.2, U17.12 (CH7), U17.19 (DGND), U17.2 (AGND), U17.3 (REFIN-), U17.9 (CH4), U18.1 (GND)
- net MDGND: now also J12.2 (Pin_2), J12.4 (Pin_4), J13.2 (Pin_2), J13.4 (Pin_4)
- net V5: now also C815.1, U18.3 (VI)
- net VIN: now also L801.4; no longer J8.1 (Pin_1)
- net VREF: now also C819.1, U17.4 (REFIN+)
- new net CS: J13.1 (Pin_1), U17.13 (CS)
- new net ENVA1: C152.1, R156.2, R157.1, U17.5 (CH0)
- new net ENVA2: C252.1, R256.2, R257.1, U17.6 (CH1)
- new net ENVA3: C352.1, R356.2, R357.1, U17.7 (CH2)
- new net ENVA4: C452.1, R456.2, R457.1, U17.8 (CH3)
- new net ENVA5: C552.1, R556.2, R557.1, U17.10 (CH5)
- new net ENVA6: C652.1, R656.2, R657.1, U17.11 (CH6)
- new net IGND_J: J8.2 (Pin_2), L801.2
- new net IRQ: J13.5 (Pin_5), U17.17 (IRQ)
- new net MCLK: J13.3 (Pin_3), U17.18 (MCLK)
- new net MISO: J12.5 (Pin_5), U17.16 (SDO)
- new net MOSI: J12.1 (Pin_1), U17.15 (SDI)
- new net SCLK: J12.3 (Pin_3), U17.14 (SCK)
- new net V3V3: C816.1, C817.1, C818.1, U17.1 (AVDD), U17.20 (DVDD), U18.2 (VO)
- new net VIN_J: J8.1 (Pin_1), L801.1
Other:
- note added: "The envelope ADC. AGND and DGND are one net here and both are MAGND -- DS20006181C section 7.3's second scheme, and the only one compatible with this board having exactly one analogue/digital star. Six logic signals leave at J12/J13 and no analogue trace crosses the boundary; MCLK is one of the six because the part's own RC oscillator cannot hold 2 kHz on six channels -- see design.envelope_adc_c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"
