File: out/cv-module.kicad_sch (KiCad schematic)
At the start: 266 parts, among them J1 CH1, J10 CTRL2, J11 CTRL3, J12 SPI, J13 SPI2, J2 CH2, J3 CH3, J4 CH4, J5 CH5, J6 CH6, J7 BOND, J8 PWR, J9 CTRL, K801 DPDT, K802 DPDT, K803 DPDT, Q801 DMG1012T, U1 OPA1644, U10 SSI2164, U11 74AHC541, U12 MAX6126A25, U13 TL074, U14 TL074, U15 TMR6-2422WI, U16 NCP1117-5.0, U17 MCP3564, U18 MCP1700-3.3, U2 OPA1644, U3 OPA1644, U4 OPA1644, U5 OPA1644, U6 OPA1644, U7 OPA1644, U8 OPA1644, U9 SSI2164

Commit message: the controller, drawn: RP2040, and DEFERRED is empty
The last deferred block. Both gates closed: the package by the fabrication
class moving to 0.09/0.09 on 1 oz (a previous pass), the supply by choosing a
part -- a TPS560430XF, and the F suffix is load-bearing.
mcu_dcdc_light_load() puts the continuous/discontinuous boundary at 91 mA
against this board's 87 mA maximum load, so a PFM part would never be
continuous and its frequency would fall to 246 kHz at idle, under the >=300 kHz
rule, on a rail the audio domain shares.

48 parts: RP2040 in QFN-56, W25Q128JV flash, ABM8-272-T3, USB micro-B at the
edge, DIN MIDI in through a TLP2761 and out through CA-033's 3.3 V pair, the
tap and expression jacks, boot/SWD headers, twelve decoupling capacitors and
the switcher. J9-J13 deleted: they were the interface to a controller on
another board.

Every value from a document read first-hand this pass -- the RP2040 datasheet,
Hardware design with RP2040, W25Q128JV rev G, TLP2761 rev 10.0, SLVSE22B,
Bourns SRN6045TA, and CA-033.

Found while drawing it, all recorded in place:

  * controller_asks() counted 14 signals across the headers that stood in for
    the block. Those carried what the *rest of the board* needed; the part also
    needs pins for its own periphery. 19 of 30.
  * the PWM row counted six carriers against sixteen *outputs*. Spec 4.2 wants
    phase stagger and a slice is one counter: six of eight.
  * supply_beat() searched twenty pump harmonics -- right for 580 kHz, the
    12.9th, and truncated at 1.1 MHz, the 24th. A fact about its only caller.
  * verify._board_copper() had never returned a single pad. Its guard read
    len(net) < 3 and every board here writes the two-element form, so
    check_isolation_gap() had been measuring tracks and vias only.
  * pad_boxes() inferred a pad's layers from its drill, and a QFN's thermal pad
    is on B.Cu as well: 64 DRC shorts from one assumption.
  * design.supply() named floorplan.check_zone_occupancy() as "the ins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
Parts:
- removed J10: CTRL2, Connector_PinHeader_2.54mm:PinHeader_1x05_P2.54mm_Vertical, symbol Connector_Generic:Conn_01x05
- removed J11: CTRL3, Connector_PinHeader_2.54mm:PinHeader_1x05_P2.54mm_Vertical, symbol Connector_Generic:Conn_01x05
- removed J12: SPI, Connector_PinHeader_2.54mm:PinHeader_1x05_P2.54mm_Vertical, symbol Connector_Generic:Conn_01x05
- removed J13: SPI2, Connector_PinHeader_2.54mm:PinHeader_1x05_P2.54mm_Vertical, symbol Connector_Generic:Conn_01x05
- removed J9: CTRL, Connector_PinHeader_2.54mm:PinHeader_1x05_P2.54mm_Vertical, symbol Connector_Generic:Conn_01x05
- added C820, C821, C822, C823, C824, C825, C826, C827, C830, C831, C834, C835, C836, C837, C838, C841, C842: 100n/50V X7R, Capacitor_SMD:C_0805_2012Metric, symbol Device:C
- added C828, C829: 1u/16V X7R, Capacitor_SMD:C_0805_2012Metric, symbol Device:C
- added C832, C833: 15p/50V C0G, Capacitor_SMD:C_0805_2012Metric, symbol Device:C
- added C840: 2u2/50V X7R, Capacitor_SMD:C_1210_3225Metric, symbol Device:C
- added C843: 22u/16V X5R, Capacitor_SMD:C_1210_3225Metric, symbol Device:C
- added D805: 1N4148W, Diode_SMD:D_SOD-123, symbol Device:D
- added J14: USB_B_Micro, Connector_USB:USB_Micro-B_Molex-105017-0001, symbol Connector:USB_B_Micro
- added J15: MIDIIN, Connector_PinHeader_2.54mm:PinHeader_1x03_P2.54mm_Vertical, symbol Connector_Generic:Conn_01x03
- added J16: MIDIOUT, Connector_PinHeader_2.54mm:PinHeader_1x03_P2.54mm_Vertical, symbol Connector_Generic:Conn_01x03
- added J17: TAP, Connector_PinHeader_2.54mm:PinHeader_1x02_P2.54mm_Vertical, symbol Connector_Generic:Conn_01x02
- added J18: EXPR, Connector_PinHeader_2.54mm:PinHeader_1x03_P2.54mm_Vertical, symbol Connector_Generic:Conn_01x03
- added J19: BOOT, Connector_PinHeader_2.54mm:PinHeader_1x03_P2.54mm_Vertical, symbol Connector_Generic:Conn_01x03
- added J20: SWD, Connector_PinHeader_2.54mm:PinHeader_1x03_P2.54mm_Vertical, symbol Connector_Generic:Conn_01x03
- added L802: 12u 20%, Inductor_SMD:L_Bourns_SRN6045TA, symbol Device:L
- added R820, R821: 27R 1%, Resistor_SMD:R_0805_2012Metric, symbol Device:R
- added R822, R823: 22k 1%, Resistor_SMD:R_0805_2012Metric, symbol Device:R
- added R824, R826, R831, R832, R833: 1k 1%, Resistor_SMD:R_0805_2012Metric, symbol Device:R
- added R825, R830: 10k 1%, Resistor_SMD:R_0805_2012Metric, symbol Device:R
- added R827: 390R 1%, Resistor_SMD:R_0805_2012Metric, symbol Device:R
- added R828: 33R 5%, Resistor_SMD:R_0805_2012Metric, symbol Device:R
- added R829: 10R 5%, Resistor_SMD:R_0805_2012Metric, symbol Device:R
- added R850: 51k 1%, Resistor_SMD:R_0805_2012Metric, symbol Device:R
- added R851: 22k1 1%, Resistor_SMD:R_0805_2012Metric, symbol Device:R
- added U19: RP2040, Package_DFN_QFN:QFN-56-1EP_7x7mm_P0.4mm_EP3.2x3.2mm_ThermalVias, symbol MCU_RaspberryPi:RP2040
- added U20: W25Q128JV, Package_SO:SOIC-8_5.3x5.3mm_P1.27mm, symbol Memory_Flash:W25Q128JVS
- added U21: TLP2761, Package_SO:SO-6L_10x3.84mm_P1.27mm, symbol Isolator:TLP2761
- added U22: TPS560430XF, Package_TO_SOT_SMD:SOT-23-6, symbol cv:TPS560430XF
- added Y801: 12MHz 30ppm, Crystal:Crystal_SMD_3225-4Pin_3.2x2.5mm, symbol Device:Crystal_GND24
Connections:
- net CS: now also U19.28 (GPIO17)
- net FSDRV: now also U19.18 (GPIO15)
- net IRQ: now also U19.31 (GPIO20)
- net MCLK: now also U19.32 (GPIO21)
- net MDGND: now also C820.2, C821.2, C822.2, C823.2, C824.2, C825.2, C826.2, C827.2, C828.2, C829.2, C830.2, C831.2, C832.2, C833.2, C834.2, C835.2, C836.2, C837.2, C838.2, C840.2, C841.2, C843.2, J14.5 (GND), J14.SH (Shield), J16.2 (Pin_2), J17.2 (Pin_2), J18.3 (Pin_3), J19.2 (Pin_2), J20.2 (Pin_2), R823.2, R851.2, U19.19 (TESTEN), U19.57 (GND), U20.4 (GND), U21.4 (GND), U22.2 (GND), Y801.2 (G), Y801.4 (G)
- net MISO: now also U19.27 (GPIO16)
- net MOSI: now also U19.30 (GPIO19)
- net OE: now also U19.17 (GPIO14)
- net PWM1: now also U19.2 (GPIO0)
- net PWM2: now also U19.4 (GPIO2)
- net PWM3: now also U19.6 (GPIO4)
- net PWM4: now also U19.8 (GPIO6)
- net PWM5: now also U19.11 (GPIO8)
- net PWM6: now also U19.13 (GPIO10)
- net SCLK: now also U19.29 (GPIO18)
- net VA_RAW: now also C840.1, C841.1, U22.4 (EN), U22.5 (VIN)
- new net BOOT: J19.1 (Pin_1), R826.2
- new net EXPR: C838.1, R833.2, U19.38 (GPIO26/ADC0)
- new net EXPRV: J18.2 (Pin_2), R832.2
- new net EXPRW: J18.1 (Pin_1), R833.1
- new net MCB: C842.1, U22.1 (CB)
- new net MFB: R850.2, R851.1, U22.3 (FB)
- new net MIDI_RX: U19.16 (GPIO13), U21.5 (VO)
- new net MIDI_TX: R829.1, U19.15 (GPIO12)
- new net MINA: D805.1 (K), R827.2, U21.1 (A)
- new net MINJ: J15.1 (Pin_1), R827.1
- new net MINK: D805.2 (A), J15.3 (Pin_3), U21.3 (K)
- new net MINSH: C836.1, J15.2 (Pin_2)
- new net MOUTD: J16.3 (Pin_3), R829.2
- new net MOUTV: J16.1 (Pin_1), R828.2
- new net MSW: C842.2, L802.1, U22.6 (SW)
- new net QSCK: U19.52 (QSPI_SCLK), U20.6 (CLK)
- new net QSCS: R826.1, U19.56 (~{QSPI_SS}), U20.1 (~{CS})
- new net QSD0: U19.53 (QSPI_SD0), U20.5 (DI/IO_{0})
- new net QSD1: U19.55 (QSPI_SD1), U20.2 (DO/IO_{1})
- new net QSD2: U19.54 (QSPI_SD2), U20.3 (~{WP}/IO_{2})
- new net QSD3: U19.51 (QSPI_SD3), U20.7 (~{HOLD}/~{RESET}/IO_{3})
- new net RUN: J19.3 (Pin_3), R825.2, U19.26 (RUN)
- new net SWCLK: J20.1 (Pin_1), U19.24 (SWCLK)
- new net SWDIO: J20.3 (Pin_3), U19.25 (SWDIO)
- new net TAP: C837.1, R831.2, U19.34 (GPIO22)
- new net TAPJ: J17.1 (Pin_1), R830.2, R831.1
- new net UDM: R820.1, U19.46 (USB_DM)
- new net UDMJ: J14.2 (D-), R820.2
- new net UDP: R821.1, U19.47 (USB_DP)
- new net UDPJ: J14.3 (D+), R821.2
- new net VBUS: J14.1 (VBUS), R822.1
- new net VBUSD: R822.2, R823.1, U19.37 (GPIO25)
- new net VCORE: C826.1, C827.1, C829.1, U19.23 (DVDD), U19.45 (VREG_VOUT), U19.50 (DVDD)
- new net VMCU: C820.1, C821.1, C822.1, C823.1, C824.1, C825.1, C828.1, C830.1, C831.1, C834.1, C835.1, C843.1, L802.2, R825.1, R828.1, R830.1, R832.1, R850.1, U19.1 (IOVDD), U19.10 (IOVDD), U19.22 (IOVDD), U19.33 (IOVDD), U19.42 (IOVDD), U19.43 (ADC_AVDD), U19.44 (VREG_VIN), U19.48 (USB_VDD), U19.49 (IOVDD), U20.8 (VCC), U21.6 (VDD)
- new net XIN: C832.1, U19.20 (XIN), Y801.1
- new net XOUT: R824.1, U19.21 (XOUT)
- new net XTAL: C833.1, R824.2, Y801.3
- no-connect marks 9 -> 22
Other:
- note added: "The controller. Two 3.3 V rails on this sheet and they are not one net: V3V3 is the ADC's, linear from V5, and VMCU is this block's, switched from VA_RAW at 1.1 MHz -- see design.RAILS. U22's input is ahead of R804 so that its ripple meets the same pole the converter's own does. MINA/MINK/MINJ are on the far side of U21 and belong to whatever is sending: CA-033 forbids a DC path from them to this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"
- note added: "The envelope ADC. AGND and DGND are one net here and both are MAGND -- DS20006181C section 7.3's second scheme, and the only one compatible with this board having exactly one analogue/digital star. Six logic signals leave for the controller and no analogue trace crosses the boundary; MCLK is one of the six because the part's own RC oscillator cannot hold 2 kHz on six channels -- see design.envelo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"
- note removed: "The envelope ADC. AGND and DGND are one net here and both are MAGND -- DS20006181C section 7.3's second scheme, and the only one compatible with this board having exactly one analogue/digital star. Six logic signals leave at J12/J13 and no analogue trace crosses the boundary; MCLK is one of the six because the part's own RC oscillator cannot hold 2 kHz on six channels -- see design.envelope_adc_c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"
