File: out/cv-module.kicad_sch (KiCad schematic)
At the start: 314 parts, among them J1 CH1, J14 USB_B_Micro, J15 MIDIIN, J16 MIDIOUT, J17 TAP, J18 EXPR, J19 BOOT, J2 CH2, J20 SWD, J3 CH3, J4 CH4, J5 CH5, J6 CH6, J7 BOND, J8 PWR, K801 DPDT, K802 DPDT, K803 DPDT, Q801 DMG1012T, U1 OPA1644, U10 SSI2164, U11 74AHC541, U12 MAX6126A25, U13 TL074, U14 TL074, U15 TMR6-2422WI, U16 NCP1117-5.0, U17 MCP3564, U18 MCP1700-3.3, U19 RP2040, U2 OPA1644, U20 W25Q128JV, U21 TLP2761, U22 TPS560430XF, U3 OPA1644, U4 OPA1644, U5 OPA1644, U6 OPA1644, U7 OPA1644, U8 OPA1644, U9 SSI2164, Y801 12MHz 30ppm

Commit message: the Pico, and the board stops being generated
The controller is a Raspberry Pi Pico -- SC0915, castellated, 2.54 mm. 314
parts and 201 nets become 289 and 184: the flash, the crystal, USB with its
terminations and VBUS divider, twelve decoupling capacitors and the BOOT and
SWD headers are all on the module.

gen_pcb.py places, pours and stitches and lays no signal copper. route.py is
deleted -- the problem it existed for went with the QFN, and what it cost was
that the board had to be a function of design.py. The netlist is generated and
authoritative; the board is hand-laid and verified. gen_pcb_guard refuses to
overwrite copper a person drew, because the pass that documented that hazard in
three files also left a run-order one-liner that triggered it.

Back-driving the module's 3V3 pin is refused on documentation rather than on
arithmetic: the RT6150 states its disconnect, its direction and its leakage,
and every one of those is stated with the input present while this needs it
absent. Feeding VSYS put two converters in series, so the 67.8 % threshold
became a threshold on a product, and the +Vout budget failed at 254.6 mA of
250. U22 moved to 5 V and took the relay coils off the linear rail -- the lever
MEASURED["mcu_dcdc_efficiency"].when_wrong had named since the QFN pass -- and
+Vout is 212.9.

The fabrication class moved three times and the round trip is the finding.
0.09/0.09 on 1 oz existed only for the QFN; 0.15/0.15 on 2 oz was derived from
the parts and omitted the 55,854 segments already on the board; and the whole
argument was against JLCPCB while the target is PCBWay, where 0.09/0.09 is not
manufacturable at any copper weight. 0.20/0.20 on 1 oz, chosen by the SOIC
corridor rather than by margin -- the coarser class has more margin and cannot
pass between two pins of a SOIC. Vias 0.7/0.3, because 0.6/0.3 was an annular
ring sitting exactly on the published minimum and nothing computed it.

Two new instruments, and each exists because nothing else would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
Parts:
- removed C820, C821, C822, C823, C824, C825, C826, C827, C830, C831, C834: 100n/50V X7R, Capacitor_SMD:C_0805_2012Metric, symbol Device:C
- removed C828, C829: 1u/16V X7R, Capacitor_SMD:C_0805_2012Metric, symbol Device:C
- removed C832, C833: 15p/50V C0G, Capacitor_SMD:C_0805_2012Metric, symbol Device:C
- removed J14: USB_B_Micro, Connector_USB:USB_Micro-B_Molex-105017-0001, symbol Connector:USB_B_Micro
- removed J20: SWD, Connector_PinHeader_2.54mm:PinHeader_1x03_P2.54mm_Vertical, symbol Connector_Generic:Conn_01x03
- removed R820, R821: 27R 1%, Resistor_SMD:R_0805_2012Metric, symbol Device:R
- removed R822, R823: 22k 1%, Resistor_SMD:R_0805_2012Metric, symbol Device:R
- removed R824, R826: 1k 1%, Resistor_SMD:R_0805_2012Metric, symbol Device:R
- removed R825: 10k 1%, Resistor_SMD:R_0805_2012Metric, symbol Device:R
- removed U20: W25Q128JV, Package_SO:SOIC-8_5.3x5.3mm_P1.27mm, symbol Memory_Flash:W25Q128JVS
- removed Y801: 12MHz 30ppm, Crystal:Crystal_SMD_3225-4Pin_3.2x2.5mm, symbol Device:Crystal_GND24
- added D806: PMEG2010AEH, Diode_SMD:D_SOD-123F, symbol Device:D_Schottky
- J19: value BOOT -> RESET; footprint Connector_PinHeader_2.54mm:PinHeader_1x03_P2.54mm_Vertical -> Connector_PinHeader_2.54mm:PinHeader_1x02_P2.54mm_Vertical; symbol Connector_Generic:Conn_01x03 -> Connector_Generic:Conn_01x02
- L802: value 12u 20% -> 15u 20%
- R850: value 51k 1% -> 88k7 1%
- U19: value RP2040 -> RaspberryPi_Pico; footprint Package_DFN_QFN:QFN-56-1EP_7x7mm_P0.4mm_EP3.2x3.2mm_ThermalVias -> Module:RaspberryPi_Pico_SMD_HandSolder; symbol MCU_RaspberryPi:RP2040 -> MCU_Module:RaspberryPi_Pico
Connections:
- net BOOT is gone; now on net RUN: J19.1 (Pin_1)
- net SWCLK is gone; now on net SCLK: U19.24 (GPIO18)
- net SWDIO is gone; now on net MOSI: U19.25 (GPIO19)
- net XIN is gone; now on net FSDRV: U19.20 (GPIO15)
- net XOUT is gone; now on net MISO: U19.21 (GPIO16)
- net CS: now also U19.22 (GPIO17); no longer U19.28 (GPIO17)
- net EXPR: now also U19.31 (GPIO26_ADC0); no longer U19.38 (GPIO26/ADC0)
- net FSDRV: no longer U19.18 (GPIO15)
- net IRQ: now also U19.26 (GPIO20); no longer U19.31 (GPIO20)
- net MCLK: now also U19.27 (GPIO21); no longer U19.32 (GPIO21)
- net MDGND: now also U19.13 (GND), U19.18 (GND), U19.23 (GND), U19.28 (GND), U19.3 (GND), U19.33 (AGND), U19.38 (GND), U19.8 (GND); no longer U19.19 (TESTEN), U19.57 (GND)
- net MIDI_RX: now also U19.17 (GPIO13); no longer U19.16 (GPIO13)
- net MIDI_TX: now also U19.16 (GPIO12); no longer U19.15 (GPIO12)
- net MISO: no longer U19.27 (GPIO16)
- net MOSI: no longer U19.30 (GPIO19)
- net OE: now also U19.19 (GPIO14); no longer U19.17 (GPIO14)
- net PWM1: now also U19.1 (GPIO0); no longer U19.2 (GPIO0)
- net PWM4: now also U19.9 (GPIO6); no longer U19.8 (GPIO6)
- net PWM6: now also U19.14 (GPIO10); no longer U19.13 (GPIO10)
- net RUN: now also U19.30 (RUN); no longer J19.3 (Pin_3), U19.26 (RUN)
- net SCLK: no longer U19.29 (GPIO18)
- net TAP: now also U19.29 (GPIO22); no longer U19.34 (GPIO22)
- net V5: no longer D813.1 (K), D823.1 (K), D833.1 (K), K801.1, K802.1, K803.1
- net VMCU: now also U19.36 (3V3); no longer C843.1, L802.2, R850.1, U19.1 (IOVDD), U19.10 (IOVDD), U19.22 (IOVDD), U19.33 (IOVDD), U19.42 (IOVDD), U19.43 (ADC_AVDD), U19.44 (VREG_VIN), U19.48 (USB_VDD), U19.49 (IOVDD)
- net VSYS: now reaches U19.39 (VSYS)
- net VSYS: now also D806.1 (K)
- removed net QSCK: U19.52 (QSPI_SCLK)
- removed net QSCS: U19.56 (~{QSPI_SS})
- removed net QSD0: U19.53 (QSPI_SD0)
- removed net QSD1: U19.55 (QSPI_SD1)
- removed net QSD2: U19.54 (QSPI_SD2)
- removed net QSD3: U19.51 (QSPI_SD3)
- removed net UDM: U19.46 (USB_DM)
- removed net UDP: U19.47 (USB_DP)
- net VBUSD: no longer names the net of U19.37 (3V3_EN)
- removed net VCORE: U19.23 (DVDD), U19.45 (VREG_VOUT), U19.50 (DVDD)
- new net VMOD: C843.1, D806.2 (A), D813.1 (K), D823.1 (K), D833.1 (K), K801.1, K802.1, K803.1, L802.2, R850.1
- no-connect marks 22 -> 21
Other:
- note added: "The controller. Three 3.3 V and 5 V nets on this sheet and no two of them are one: V3V3 is the ADC's, linear from V5; VMOD is U22's switched 5 V, carrying the module and the relay coils; VMCU is the module's own 3.3 V, made on it by an RT6150 out of VSYS and brought back out on pin 36. V5 is what is left of the linear rail -- the reference and the ADC's LDO. U22's input is ahead of R804 so that i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"
- note removed: "The controller. Two 3.3 V rails on this sheet and they are not one net: V3V3 is the ADC's, linear from V5, and VMCU is this block's, switched from VA_RAW at 1.1 MHz -- see design.RAILS. U22's input is ahead of R804 so that its ripple meets the same pole the converter's own does. MINA/MINK/MINJ are on the far side of U21 and belong to whatever is sending: CA-033 forbids a DC path from them to this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"

Commit message: the placement closes at zero, the fuse is fitted, and the board is seeded
Four things this pass, and the last one found five more.

**placement.check_courtyard_gap() is 0, from 23.** Two functions replace the
nudging that took 41 to 23 and then to 12-with-three-overlaps: pack_east()
lays a row west to east at required_gap(), and clear_south() stacks the seven
bands south of the relays, each naming the one pair that sets it. The pair is
a claim, not an assertion -- the gap check walks all 290 parts, so a band
derived from the wrong neighbour fails and says which pair it should have
been. It earned that within the hour. Cost: 3.6 mm of length, 1.7 of width.

**The inlet fuse is fitted.** SCHURTER UMT 250, 1.6 A time-lag, 3403.0168.11,
datasheet and DigiKey page both read. The requirement never moved; the blocker
was one manufacturer's catalogue written as a fact about the part class. 1.6 A
and not the derived 1.5, because 1.5 is not an IEC 60127 step. inlet_budget()'s
series resistance gained three names, because the moment the fuse joined the
loop `choke_r` stopped being the choke's.

**The hole rules are owned, and the open question had the wrong page's number
in it.** It asked whether to take JLCPCB's 0.20 mm over KiCad's 0.25 -- on a
PCBWay board. PCBWay publishes 0.406 hole-to-hole and 0.178 hole-to-copper, so
the fabricator is stricter on one and looser on the other. rules.hole_rules()
takes the stricter of published and KiCad's for each; neither binds, because
copper sets all three of a via's distances at this class.

**route.py is restored and ran once.** --seed-routing, so what is handed over
is a legal route to adjust rather than 486 airwires. Nothing in the file
changed to come back. It closed every net: 1652 tracks, 595 vias, 151 stitches,
0 unconnected, 0 DRC, and check_board_is_the_design() passes for the first
time. UNROUTED_ITEMS is 0 and stays a ratchet.

What the seed found, none of it visible to anything else here:

  * EDGE_PARTS declares a side an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
Parts:
- added F801: 1.6A T 250V, Fuse:Fuse_Schurter_UMT250, symbol Device:Fuse
Connections:
- net VIN_J: now also F801.1; no longer L801.1
- new net VIN_F: F801.2, L801.1
Changed lines of the file:
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@@
 	(wire
 		(pts
+			(xy 68.58 1092.2)
+			(xy 60.96 1092.2)
+		)
+		(stroke
+			(width 0)
+			(type default)
+		)
+	)
+	(wire
+		(pts
+			(xy 76.2 1092.2)
+			(xy 83.82 1092.2)
+		)
+		(stroke
+			(width 0)
+			(type default)
+		)
+	)
+	(wire
+		(pts
 			(xy 90.17 1089.66)
 			(xy 82.55 1089.66)
@@
 	(global_label "VIN_J"
 		(shape input)
+		(at 60.96 1092.2 0)
+		(effects
+			(font
+				(size 1.27 1.27)
+			)
+			(justify left)
+		)
+	)
+	(global_label "VIN_F"
+		(shape input)
+		(at 83.82 1092.2 0)
+		(effects
+			(font
+				(size 1.27 1.27)
+			)
+			(justify left)
+		)
+	)
+	(global_label "VIN_F"
+		(shape input)
 		(at 82.55 1089.66 0)
 		(effects
@@
 					(unit 1)
 				)
+			)
+		)
+	)
+	(symbol
+		(lib_id "Device:Fuse")
+		(at 72.39 1092.2 90)
+		(unit 1)
+		(exclude_from_sim no)
+		(in_bom yes)
+		(on_board yes)
+		(dnp no)
+		(property "Reference" "F801"
+			(at 72.39 1085.85 0)
+			(effects
+				(font
+					(size 1.27 1.27)
+				)
+				(justify left)
+			)
+		)
+		(property "Value" "1.6A T 250V"
+			(at 72.39 1098.55 0)
+			(effects
+				(font
+					(size 1.27 1.27)
+				)
+				(justify left)
+			)
+		)
+		(property "Footprint" "Fuse:Fuse_Schurter_UMT250"
+			(at 72.39 1092.2 0)
+			(effects
+				(font
+					(size 0.762 0.762)
+				)
+				(hide yes)
+			)
+		)
+		(property "Datasheet" "~"
+			(at 72.39 1092.2 0)
+			(effects
+				(font
+					(size 1.27 1.27)
+				)
+				(hide yes)
+			)
+		)
+		(pin "1"
+		)
+		(pin "2"
+		)
+		(instances
+			(project "cv-module"
+				(path "/234c64a2-6120-5e9c-89d1-a2d4cf0dfab9"
+					(reference "F801")
+					(unit 1)
+				)

Commit message: DC bias modelled from the manufacturers' own curves, and two parts changed
Run before Tim starts routing, to find out whether any capacitor needs a
different land. **None does.** Both parts that changed keep their 1210
footprint and differ only in body height, so the board is safe to route.

**Nothing here modelled DC bias.** Every ceramic was declared at zero volts
and used as though that were its value in circuit -- RAIL_FILTER_ESR's shape
exactly: not a wrong number, a number computed without the term that
dominates. CAP_DC_BIAS holds the manufacturers' own characterisation, read
off TDK's product pages, not a per-class rule of thumb: derating is specific
to a part number and a table of typical percentages by case size is the
invented constant section 6 forbids.

**C840 was 25 % short of a stated minimum.** CGA6M3X7R1H225K200AB holds
1.65 uF of its 2.2 at the 12 V it sits at, against TI 9.2.2.6's "2.2 uF or
higher" -- four times the part's own tolerance, so not a tolerance question.
Now CGA6P3X7R1H475K250AB, a 4.7 uF part holding **4.23 uF at 12 V**, 1.9x the
requirement. Same 1210 land, 2.5 mm tall instead of 2.0.

The first candidate for that swap, CGA6M3X7R1H475K200AB, returned a 404 on
TDK's site. Guess-and-verify is fine; guess-and-assert is what produced an
invented part number earlier in this repo's week.

**And the 10 uF 50 V line was quietly uncharacterised.** Murata's SimSurfing
answers "The specified partnumber not exist" for GRM32ER71H106KA12L while
returning 7 kB for its 63 V sibling. Distributors still hold stock, so the
part is not fictional -- what is gone is the manufacturer's characterisation,
which normally means legacy, and it is why no bias curve could be had for the
five capacitors that sit at 12 to 20 V.

Replaced with **CNA6P1X7R1H106K250AE**: TDK, AEC-Q200, soft termination,
50 VDC so the value string does not move and nobody can substitute a 50 V
part back in against a 63 V line. 1210, 2.5 mm tall, in Production. It holds
7.89 uF at 12 V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
Parts:
- C801: value 100n/50V C0G -> 100n/50V X7R
- C840: value 2u2/50V X7R -> 4u7/50V X7R
Changed lines of the file:
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@@
 			)
 		)
-		(property "Value" "100n/50V C0G"
+		(property "Value" "100n/50V X7R"
 			(at 25.4 793.75 0)
 			(effects
@@
 			)
 		)
-		(property "Value" "2u2/50V X7R"
+		(property "Value" "4u7/50V X7R"
 			(at 762 1536.7 0)
 			(effects

Commit message: the board carries the right lands now, and the sync cost four things
The design fix was three part numbers and one footprint. Putting it on the board
took a re-route, a stitch via, a rule change and a corrected command, and none of
those was on the list. docs/footprint-audit.md records all four.

The re-route scope had to be derived rather than guessed. Moving five diodes from
a two-pad land to a three-pad one puts their pads under other nets' copper: DRC
named MISO, IRQ, MOSI and PWM5 alongside the four nets the diodes are on, so the
scope came off the report -- FSAC FSG FSD VMOD MISO IRQ MOSI PWM5 -- which is
krt.plan()'s own rescue rule arriving in a scoped run. 71 violations and 10
unconnected items became 12 and 0.

And --nets takes patterns, not a comma-separated list. "FSAC,FSG,FSD,VMOD" is one
pattern matching nothing, and route.py refuses with "none of the 1 requested net
name(s) exist on this board" rather than routing nothing quietly.

MDGND was excluded from the scope and had to be -- its 35 segments on the signal
layers are stitch_grounds()' stubs to the plane, not routing -- so D801's anode
was left open and the router's improvement gate refused to commit, correctly:
disconnected_pads_before 10, after 1, and the 1 was that pad. Its old stitch ran
east from a pad that has moved, and KiCad re-netted that via to FSAC when the new
cathode pad landed on it, which is why DRC reported a via at 0.0000 mm against
the MDGND pour. A via and a stub at (42.35, 168.0775), 0.76 mm from the pad and
clear of the body, chosen by searching the candidate board for a position legal
against the class rules -- the same geometry stitch_grounds() lays 151 times.

The last twelve violations were silkscreen and came from a rule reading a proxy.
gen_pcb.py puts a designator on F.Fab rather than silk when a part has two pads,
because 128 parts here are smaller than their own reference text. A SOT-23 has
three pads -- the middle one is not connected -- so the rule stopped applying,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
Parts:
- D801, D802, D813, D823, D833: footprint Diode_SMD:D_SOD-123 -> Package_TO_SOT_SMD:SOT-23; symbol Device:D -> cv:BAT54
Connections:
- net FSAC: now also D801.3 (K), D802.1 (A); no longer D801.1 (K), D802.2 (A)
- net FSD: now also D813.1 (A), D823.1 (A), D833.1 (A); no longer D813.2 (A), D823.2 (A), D833.2 (A)
- net FSG: now also D802.3 (K); no longer D802.1 (K)
- net MDGND: now also D801.1 (A); no longer D801.2 (A)
- net VMOD: now also D813.3 (K), D823.3 (K), D833.3 (K); no longer D813.1 (K), D823.1 (K), D833.1 (K)
Changed lines of the file:
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@@
 	)
 	(symbol
-		(lib_id "Device:D")
+		(lib_id "cv:BAT54")
 		(at 889 949.96 90)
 		(unit 1)
@@
 			)
 		)
-		(property "Footprint" "Diode_SMD:D_SOD-123"
+		(property "Footprint" "Package_TO_SOT_SMD:SOT-23"
 			(at 889 949.96 0)
 			(effects
@@
 		(pin "1"
 		)
-		(pin "2"
+		(pin "3"
 		)
 		(instances
@@
 	)
 	(symbol
-		(lib_id "Device:D")
+		(lib_id "cv:BAT54")
 		(at 889 929.64 90)
 		(unit 1)
@@
 			)
 		)
-		(property "Footprint" "Diode_SMD:D_SOD-123"
+		(property "Footprint" "Package_TO_SOT_SMD:SOT-23"
 			(at 889 929.64 0)
 			(effects
@@
 		(pin "1"
 		)
-		(pin "2"
+		(pin "3"
 		)
 		(instances
@@
 	)
 	(symbol
-		(lib_id "Device:D")
+		(lib_id "cv:BAT54")
 		(at 812.8 1016 90)
 		(unit 1)
@@
 			)
 		)
-		(property "Footprint" "Diode_SMD:D_SOD-123"
+		(property "Footprint" "Package_TO_SOT_SMD:SOT-23"
 			(at 812.8 1016 0)
 			(effects
@@
 		(pin "1"
 		)
-		(pin "2"
+		(pin "3"
 		)
 		(instances
@@
 	)
 	(symbol
-		(lib_id "Device:D")
+		(lib_id "cv:BAT54")
 		(at 863.6 1016 90)
 		(unit 1)
@@
 			)
 		)
-		(property "Footprint" "Diode_SMD:D_SOD-123"
+		(property "Footprint" "Package_TO_SOT_SMD:SOT-23"
 			(at 863.6 1016 0)
 			(effects
@@
 		(pin "1"
 		)
-		(pin "2"
+		(pin "3"
 		)
 		(instances
@@
 	)
 	(symbol
-		(lib_id "Device:D")
+		(lib_id "cv:BAT54")
 		(at 914.4 1016 90)
 		(unit 1)
@@
 			)
 		)
-		(property "Footprint" "Diode_SMD:D_SOD-123"
+		(property "Footprint" "Package_TO_SOT_SMD:SOT-23"
 			(at 914.4 1016 0)
 			(effects
@@
 		(pin "1"
 		)
-		(pin "2"
-		)
-		(instances
+		(pin "3"
+		)
+		(instances
