File: out/cv-module.kicad_pcb (KiCad board)
At the start: 4 copper layers, 106.9 x 233.6 mm, 290 parts, among them J1 CH1, J15 MIDIIN, J16 MIDIOUT, J17 TAP, J18 EXPR, J19 RESET, J2 CH2, J3 CH3, J4 CH4, J5 CH5, J6 CH6, J7 BOND, J8 PWR, K801 G6S-2 DC5, K802 G6S-2 DC5, K803 G6S-2 DC5, Q801 DMG1012T, U1 OPA1644, U10 SSI2164, U11 74AHC541, U12 MAX6126A25, U13 TL074, U14 TL074, U15 TMR6-2422WI, U16 NCP1117-5.0, U17 MCP3564, U18 MCP1700-3.3, U19 RaspberryPi_Pico, U2 OPA1644, U21 TLP2761, U22 TPS560430XF, U3 OPA1644, U4 OPA1644, U5 OPA1644, U6 OPA1644, U7 OPA1644, U8 OPA1644, U9 SSI2164

Commit message: DC bias modelled from the manufacturers' own curves, and two parts changed
Run before Tim starts routing, to find out whether any capacitor needs a
different land. **None does.** Both parts that changed keep their 1210
footprint and differ only in body height, so the board is safe to route.

**Nothing here modelled DC bias.** Every ceramic was declared at zero volts
and used as though that were its value in circuit -- RAIL_FILTER_ESR's shape
exactly: not a wrong number, a number computed without the term that
dominates. CAP_DC_BIAS holds the manufacturers' own characterisation, read
off TDK's product pages, not a per-class rule of thumb: derating is specific
to a part number and a table of typical percentages by case size is the
invented constant section 6 forbids.

**C840 was 25 % short of a stated minimum.** CGA6M3X7R1H225K200AB holds
1.65 uF of its 2.2 at the 12 V it sits at, against TI 9.2.2.6's "2.2 uF or
higher" -- four times the part's own tolerance, so not a tolerance question.
Now CGA6P3X7R1H475K250AB, a 4.7 uF part holding **4.23 uF at 12 V**, 1.9x the
requirement. Same 1210 land, 2.5 mm tall instead of 2.0.

The first candidate for that swap, CGA6M3X7R1H475K200AB, returned a 404 on
TDK's site. Guess-and-verify is fine; guess-and-assert is what produced an
invented part number earlier in this repo's week.

**And the 10 uF 50 V line was quietly uncharacterised.** Murata's SimSurfing
answers "The specified partnumber not exist" for GRM32ER71H106KA12L while
returning 7 kB for its 63 V sibling. Distributors still hold stock, so the
part is not fictional -- what is gone is the manufacturer's characterisation,
which normally means legacy, and it is why no bias curve could be had for the
five capacitors that sit at 12 to 20 V.

Replaced with **CNA6P1X7R1H106K250AE**: TDK, AEC-Q200, soft termination,
50 VDC so the value string does not move and nobody can substitute a 50 V
part back in against a 63 V line. 1210, 2.5 mm tall, in Production. It holds
7.89 uF at 12 V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
Parts:
- C801: value 100n/50V C0G -> 100n/50V X7R
- C840: value 2u2/50V X7R -> 4u7/50V X7R
